File: Actuators Board/power.sch (KiCad schematic (older format))
At the start: 32 parts, among them J11 Conn_01x02_Male, U12 MAX40200AUK, U8 TPS63031

Commit message: usbc completed and autoboot fixed
Parts:
- U8: symbol Mainboard-rescue:TPS63031-iclr -> Mainboard-rescue:TPS63031-iclr-Mainboard-rescue
Changed lines of the file:
@@
 	3800 5150 4100 5150
 $Comp
-L Mainboard-rescue:+3.3V-Mainboard-cache #PWR0106
+L Mainboard-rescue:+3.3V-Mainboard-cache-Mainboard-rescue #PWR0106
 U 1 1 5E4CE71E
 P 3800 5150
@@
 $EndComp
 $Comp
-L Mainboard-rescue:TPS63031-iclr U8
+L Mainboard-rescue:TPS63031-iclr-Mainboard-rescue U8
 U 1 1 5DE04FA4
 P 5900 4000
