File: Actuators Board/board_template.sch (KiCad schematic (older format))
At the start: 27 parts, among them J10 Conn_01x02_Male, J9 Conn_01x02_Male, Q1 MMDT2222A

Commit message: Place Hierarchical Pins from CAN sheet to each board.
Changed lines of the file:
@@
 F0 "CAN-BUS" 50
 F1 "can.sch" 50
+F2 "CAN_TX" O R 4600 6850 50
+F3 "CAN_RX" I R 4600 6950 50
 $EndSheet
 Text Label 5000 2150 0    50   ~ 0
@@
 Text Label 4750 850  2    50   ~ 0
 LNA_IN
+Wire Wire Line
+	4600 6850 4700 6850
+Text Label 4700 6850 0    50   ~ 0
+CAN_TX
+Text Label 4700 6950 0    50   ~ 0
+CAN_RX
+Wire Wire Line
+	4600 6950 4700 6950
 $EndSCHEMATC

Commit message: Connected 3.3V to ESP32 according to schematic
Parts:
- added C?: 10uF, symbol Device:C_Small
- added C?: 0.1uF, symbol Device:C_Small
Connections:
- net +3V3: now also U?.1 (VDDA), U?.19 (VDD3P3_RTC), U?.37 (VDD3P3_CPU), U?.43 (VDDA), U?.46 (VDDA), C?.1, C?.1
- net GND: now also C?.2, C?.2
Changed lines of the file:
@@
 $EndDescr
-$Comp
-L power:+3.3V #PWR020
-U 1 1 5DA60792
-P 4100 1950
-F 0 "#PWR020" H 4100 1800 50  0001 C CNN
-F 1 "+3.3V" H 4115 2123 50  0000 C CNN
-F 2 "" H 4100 1950 50  0001 C CNN
-F 3 "" H 4100 1950 50  0001 C CNN
-	1    4100 1950
-	1    0    0    -1
-$EndComp
 $Comp
 L power:GND #PWR021
@@
 LNA_IN
 $Sheet
-S 4950 750  1750 400
+S 5950 700  1750 400
 U 61A49DAE
 F0 "rfantenna" 50
 F1 "rfantenna.sch" 50
-F2 "LNA_IN" B L 4950 850 50
+F2 "LNA_IN" B L 5950 800 50
 $EndSheet
 Wire Wire Line
-	4950 850  4750 850
-Text Label 4750 850  2    50   ~ 0
+	5950 800  5750 800
+Text Label 5750 800  2    50   ~ 0
 LNA_IN
 Wire Wire Line
@@
 Wire Wire Line
 	4600 6950 4700 6950
+$Comp
+L power:+3.3V #PWR?
+U 1 1 61A739D1
+P 3600 1800
+F 0 "#PWR?" H 3600 1650 50  0001 C CNN
+F 1 "+3.3V" H 3615 1973 50  0000 C CNN
+F 2 "" H 3600 1800 50  0001 C CNN
+F 3 "" H 3600 1800 50  0001 C CNN
+	1    3600 1800
+	-1   0    0    1
+$EndComp
+$Comp
+L Device:C_Small C?
+U 1 1 61A75CFA
+P 3700 1700
+F 0 "C?" H 3500 1750 50  0000 L CNN
+F 1 "10uF" H 3450 1650 50  0000 L CNN
+F 2 "" H 3700 1700 50  0001 C CNN
+F 3 "~" H 3700 1700 50  0001 C CNN
+	1    3700 1700
+	-1   0    0    1
+$EndComp
+$Comp
+L Device:C_Small C?
+U 1 1 61A79B6C
+P 3500 1700
+F 0 "C?" H 3592 1746 50  0000 L CNN
+F 1 "0.1uF" H 3592 1655 50  0000 L CNN
+F 2 "" H 3500 1700 50  0001 C CNN
+F 3 "~" H 3500 1700 50  0001 C CNN
+	1    3500 1700
+	-1   0    0    1
+$EndComp
+Wire Wire Line
+	3700 1800 3600 1800
+Wire Wire Line
+	3700 1600 3600 1600
+$Comp
+L power:GND #PWR?
+U 1 1 61A8986C
+P 3600 1600
+F 0 "#PWR?" H 3600 1350 50  0001 C CNN
+F 1 "GND" H 3605 1427 50  0000 C CNN
+F 2 "" H 3600 1600 50  0001 C CNN
+F 3 "" H 3600 1600 50  0001 C CNN
+	1    3600 1600
+	-1   0    0    1
+$EndComp
+Connection ~ 3600 1600
+Wire Wire Line
+	3600 1600 3500 1600
+Connection ~ 3600 1800
+Wire Wire Line
+	3600 1800 3500 1800
+Wire Wire Line
+	4000 1900 4100 1900
+Wire Wire Line
+	4100 1900 4100 1950
+Wire Wire Line
+	4000 1900 4000 1950
+Wire Wire Line
+	4100 1900 4200 1900
+Wire Wire Line
+	4200 1900 4200 1950
+Connection ~ 4100 1900
+Wire Wire Line
+	4200 1900 4300 1900
+Wire Wire Line
+	4300 1900 4300 1950
+Connection ~ 4200 1900
+Wire Wire Line
+	3700 1800 4000 1800
+Wire Wire Line
+	4000 1800 4000 1900
+Connection ~ 3700 1800
+Connection ~ 4000 1900
 $EndSCHEMATC

Commit message: Connected 3.3V output from USB-UART converter
Changed lines of the file:
@@
 F4 "TXD" O R 2200 3450 50
 F5 "DTR" O R 2200 3550 50
+F6 "3.3V" O R 2200 3650 50
 $EndSheet
 $Comp
@@
 Connection ~ 3700 1800
 Connection ~ 4000 1900
+Wire Wire Line
+	2200 3650 2300 3650
+$Comp
+L power:+3.3V #PWR?
+U 1 1 61A6C8AA
+P 2300 3650
+F 0 "#PWR?" H 2300 3500 50  0001 C CNN
+F 1 "+3.3V" V 2315 3778 50  0000 L CNN
+F 2 "" H 2300 3650 50  0001 C CNN
+F 3 "" H 2300 3650 50  0001 C CNN
+	1    2300 3650
+	0    1    1    0
+$EndComp
 $EndSCHEMATC

Commit message: Added main connector, CAN hierarchical pins and changed LEDs on template
Parts:
- removed D17: USB_LED, LED_SMD:LED_0603_1608Metric_Castellated, symbol Device:LED_Small
- removed D2: RX_LED, LED_SMD:LED_0603_1608Metric_Castellated, symbol Device:LED_Small
- removed D3: TX_LED, LED_SMD:LED_0603_1608Metric_Castellated, symbol Device:LED_Small
- removed D6: PWR_LED, LED_SMD:LED_0603_1608Metric_Castellated, symbol Device:LED_Small
- removed R10, R11, R14, R36: 470, Resistor_SMD:R_0603_1608Metric, symbol Device:R_Small
- added D?: TX_LED, LED_SMD:LED_0603_1608Metric_Castellated, symbol Device:LED_Small
- added D?: RX_LED, LED_SMD:LED_0603_1608Metric_Castellated, symbol Device:LED_Small
- added D?: 3.3V LED, LED_SMD:LED_0603_1608Metric_Castellated, symbol Device:LED_Small
- added D?: 24V LED, LED_SMD:LED_0603_1608Metric_Castellated, symbol Device:LED_Small
- added J?: Conn_01x05_Male, symbol Connector:Conn_01x05_Male
- added R? (x5): 470, Resistor_SMD:R_0603_1608Metric, symbol Device:R_Small
- added R? (x2): 1k, Resistor_SMD:R_0603_1608Metric, symbol Device:R_Small
Connections:
- net +3V3: now also J?.3 (Pin_3), R?.1, R?.1, R?.2
- net GND: now also D?.1 (K), D?.1 (K), J?.4 (Pin_4), R?.1, R?.1, R?.2, R?.2
- net RXD: now also D?.1 (K)
- net TXD: now also D?.1 (K)
- new net: D?.2 (A), R?.2 (x2)
- new net: D?.2 (A), R?.1 (x2)
- new net: R?.1, R?.2
- new net +24V: J?.5 (Pin_5), R?.2
- new net CAN_HIGH: J?.2 (Pin_2)
- new net CAN_LOW: J?.1 (Pin_1)
