File: Actuators Board/rfantenna.kicad_sch (KiCad schematic)
At the start: 4 parts

Commit message: autoboot circuit layout
Parts:
- L1: footprint Inductor_SMD:L_0402_1005Metric_Pad0.77x0.64mm_HandSolder -> Inductor_SMD:L_0603_1608Metric_Pad1.05x0.95mm_HandSolder
Changed lines of the file:
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@@
     (property "Reference" "L1" (id 0) (at 148.59 37.084 90))
     (property "Value" "LQG15WZ1N8B02D" (id 1) (at 148.59 39.3954 90))
-    (property "Footprint" "Inductor_SMD:L_0402_1005Metric_Pad0.77x0.64mm_HandSolder" (id 2) (at 148.59 41.91 0)
+    (property "Footprint" "Inductor_SMD:L_0603_1608Metric_Pad1.05x0.95mm_HandSolder" (id 2) (at 148.59 41.91 0)
       (effects (font (size 1.27 1.27)) hide)
     )
