File: Actuators Board/Actuators Board - Copy.kicad_sch (KiCad schematic)
At the start: 73 parts, among them J1 Conn_01x05_Male, J10 Conn_01x02_Male, J2 Solenoid(Sol), J4 Conn_01x03_Male, J5 Conn_01x06_Male, J9 Conn_01x02_Male, Q1 MMDT2222A, Q2 SI2366DS, U1 ESP32-PICO-D4, U2 TPS54233D, U5 MAX14871EUE+

Commit message: copied files and fixed usb
Parts:
- removed C14: 10uF, Capacitor_SMD:C_0603_1608Metric, symbol Device:CP1_Small
- removed C18: 10uF, Capacitor_SMD:C_0603_1608Metric, symbol Device:C_Small
- removed C20: 100uF, Capacitor_SMD:C_0603_1608Metric, symbol Device:C_Small
- removed D9: D, Diode_SMD:D_0603_1608Metric_Castellated, symbol Device:D
- removed R13: 10k, Resistor_SMD:R_0603_1608Metric, symbol Device:R_Small
- removed R3: 470, Resistor_SMD:R_0603_1608Metric, symbol Device:R_Small
- removed R6: 1k, Resistor_SMD:R_0603_1608Metric, symbol Device:R_Small
- removed R_SENS1: 0.1, Resistor_SMD:R_0603_1608Metric, symbol Device:R_Small
- removed TP22: TestPoint, TestPoint:TestPoint_THTPad_1.0x1.0mm_Drill0.5mm, symbol Connector:TestPoint
- removed U5: MAX14871EUE+, iclr:SOP65P637X110-16N, symbol iclr:MAX14871EUE+
- added C14, C7: 10uF, Capacitor_SMD:C_1210_3225Metric, symbol Device:C_Small
- added C22: 4.7uF, Capacitor_SMD:C_0603_1608Metric, symbol Device:C_Small
- added D11, D12, D9: V8PAM10S, iclr:DIO_V3PAN50-M3_I, symbol iclr:V3PAN50-M3{brace}slash}I
- added IC1: BD62120AEFJ-E2, iclr:SOIC127P600X100-9N, symbol iclr:BD62120AEFJ-E2
- added U5: LTC4411, Package_TO_SOT_SMD:SOT-23-5, symbol iclr:LTC4411
- C1, C3: value 0.1uF -> 1uF
- C17: value 1uF -> 0.1uF
- C19: value 470uF -> 100uF; footprint Capacitor_SMD:CP_Elec_8x6.7 -> Capacitor_SMD:CP_Elec_5x5.9
- D1, D2, D3, D6, D7: footprint LED_SMD:LED_0603_1608Metric_Castellated -> LED_SMD:LED_0603_1608Metric
- D8: value B340 -> MBR260HWTR; footprint Diode_SMD:D_SMC -> Diode_SMD:D_SOD-123
- J1: footprint Connector_PinHeader_2.54mm:PinHeader_1x05_P2.54mm_Vertical -> (none)
- J4: footprint Connector_PinHeader_2.54mm:PinHeader_1x03_P2.54mm_Vertical -> Connector_JST:JST_XH_B3B-XH-AM_1x03_P2.50mm_Vertical
- L2: value PE-92111KNL -> ETQP5M; footprint Inductor_SMD:L_12x12mm_H6mm -> iclr:IND_ETQP5M330YFM
- R12: value 1k -> 10k
- R4: value 470 -> 3.5k
Connections:
- net +24V: now also J1.3 (Pin_3), R4.1, C14.1, C7.1, D9.C, IC1.3 (VCC); no longer J1.5 (Pin_5), R12.1
- net +3V3: now also C22.1, U5.5 (OUT); no longer J1.4 (Pin_4)
- net CAN_HIGH: now also J1.1 (Pin_1); no longer J1.2 (Pin_2)
- net CAN_LOW: now also J1.5 (Pin_5); no longer J1.1 (Pin_1)
- net GND: now also J1.2 (Pin_2), R12.2, C14.2, C22.2, C7.2, D11.A, D12.A, IC1.1 (GND_1), IC1.4 (GND_2), IC1.7 (TEST), IC1.9 (EP), U5.2 (GND), U5.3 (CTL); no longer J1.3 (Pin_3), R21.2
- net Motor+: now also D12.C, IC1.8 (OUT2)
- net Motor-: now also D11.C, IC1.2 (OUT1)
- net ServoPWM: now also U1.17 (IO14); no longer U1.20 (IO13)
- net SolEN: now also R12.1, R21.2, U1.21 (IO15); no longer Q2.1 (G), R21.1, U1.18 (IO12)
- net SolGND: now also D9.A
- net HBridgeDIR renamed HBridgeDIR1
- net HBridgeDIR1: now also IC1.5 (IN1)
- net HBridgePWM renamed HBridgeDIR2
- net HBridgeDIR2: now also IC1.6 (IN2)
- new net: J1.4 (Pin_4), U5.1 (IN)
- new net: Q2.1 (G), R21.1
Other:
- moved on the sheet: J1, J2, J4, R21

Commit message: SOL and U5 connections added
copies of the files also made. Connections are about the bottom and U5 is at the right side.
Parts:
- removed D11, D12, D9: V8PAM10S, iclr:DIO_V3PAN50-M3_I, symbol iclr:V3PAN50-M3{brace}slash}I
- removed TP12, TP13, TP15, TP2, TP3: TestPoint, TestPoint:TestPoint_THTPad_1.0x1.0mm_Drill0.5mm, symbol Connector:TestPoint
- added D10, D11, D9: V8PAM10S, iclr:DIO_V3PAN50-M3_I, symbol iclr:V8PAM10S
- added H1, H2, H3, H4: MountingHole_Pad, MountingHole:MountingHole_3.2mm_M3_DIN965_Pad, symbol Mechanical:MountingHole_Pad
- added R13: 470, Resistor_SMD:R_0603_1608Metric, symbol Device:R_Small
- J5: footprint Connector_PinSocket_2.54mm:PinSocket_1x06_P2.54mm_Vertical -> Connector_PinHeader_2.54mm:PinHeader_1x06_P2.54mm_Vertical
Connections:
- net +24V: now also D9.C
- net CAN_RX: now also U1.16 (IO27); no longer U1.13 (IO33)
- net CAN_TX: now also U1.17 (IO14); no longer U1.12 (IO32)
- net GND: now also D10.A, D11.A, H1.1, H2.1, H3.1, H4.1
- net HBridgeDIR2: now also U1.14 (IO25); no longer U1.16 (IO27)
- net Hall1: now also U1.10 (IO34); no longer U1.34 (IO5)
- net Hall2: now also U1.11 (IO35); no longer U1.24 (IO4)
- net Motor+: now also D11.C
- net Motor-: now also D10.C
- net ServoPWM: now also U1.13 (IO33); no longer U1.17 (IO14)
- net SolEN: now also U1.12 (IO32), R13.2; no longer D1.2 (A), U1.21 (IO15)
- net SolGND: now also D9.A
- new net: D1.2 (A), R13.1
Other:
- moved on the sheet: D1, TP14, TP16, TP20, TP21, TP4

Commit message: most of board copy sorted
Parts:
- removed TP8: TestPoint, TestPoint:TestPoint_THTPad_1.0x1.0mm_Drill0.5mm, symbol Connector:TestPoint
- added C26: 100pF, Capacitor_SMD:C_0603_1608Metric, symbol Device:C_Small
- added C27: 10uF, Capacitor_SMD:C_0603_1608Metric, symbol Device:C_Small
- added C28: 1uF, Capacitor_SMD:C_0603_1608Metric, symbol Device:C_Small
- added C29, C30, C31: 0.1uF, Capacitor_SMD:C_0603_1608Metric, symbol Device:C_Small
- added JP1: SolderJumper_2_Open, Jumper:SolderJumper-2_P1.3mm_Open_RoundedPad1.0x1.5mm, symbol Jumper:SolderJumper_2_Open
- added TP12, TP2, TP3: TestPoint, TestPoint:TestPoint_THTPad_1.0x1.0mm_Drill0.5mm, symbol Connector:TestPoint
- C4: value 10uF -> 0.1uF
- C5: value 0.1uF -> 1uF
- J1: footprint (none) -> Connector_PinHeader_2.54mm:PinHeader_1x05_P2.54mm_Vertical
- J2: footprint (none) -> Connector_PinHeader_2.54mm:PinHeader_1x02_P2.54mm_Vertical
- TP20, TP21, TP6, TP7: footprint TestPoint:TestPoint_THTPad_1.0x1.0mm_Drill0.5mm -> TestPoint:TestPoint_Pad_D1.0mm
- U2: footprint iclr:SOIC127P599X175-8N -> Package_SO:SOIC-8-1EP_3.9x4.9mm_P1.27mm_EP2.29x3mm_ThermalVias
Connections:
- net +24V: now also JP1.2 (B)
- net +3V3: now also C4.1, C26.1, C27.1, C28.1, C29.1, C30.1, C31.1; no longer C4.2
- net +6V: now also JP1.1 (A)
- net GND: now also C4.2, U2.9 (GND), C26.2, C27.2, C28.2, C29.2, C30.2, C31.2; no longer C4.1
- net Hall1: now also U1.12 (IO32), TP3.1; no longer U1.10 (IO34)
- net Hall2: now also TP2.1
- net Motor+: now also IC1.2 (OUT1); no longer IC1.8 (OUT2)
- net Motor-: now also IC1.8 (OUT2); no longer IC1.2 (OUT1)
- net ServoPWM: now also U1.10 (IO34), TP12.1; no longer U1.13 (IO33)
- net SolEN: now also U1.34 (IO5); no longer U1.12 (IO32)
Other:
- note added: "Pin 1"
- note added: "Pin 43"
- note added: "Pin 46"
- moved on the sheet: C14, TP14, TP23
