File: Chad/Hardware/rfantenna.kicad_sch (KiCad schematic)
At the start: 4 parts

Commit message: Implemented design review feedback
Parts:
- C11: value 1.2pF -> 33pF
- C12: value 1.5pF -> 100pF
Changed lines of the file:
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@@
       (effects (font (size 1.27 1.27)) (justify left))
     )
-    (property "Value" "1.5pF" (id 1) (at 154.7368 48.133 0)
+    (property "Value" "100pF" (id 1) (at 154.7368 48.133 0)
       (effects (font (size 1.27 1.27)) (justify left))
     )
@@
       (effects (font (size 1.27 1.27)) (justify left))
     )
-    (property "Value" "1.2pF" (id 1) (at 137.16 48.26 0)
+    (property "Value" "33pF" (id 1) (at 137.16 48.26 0)
       (effects (font (size 1.27 1.27)) (justify left))
     )
