File: Chad/Hardware/Actuators Board.kicad_pcb (KiCad board)
At the start: 4 copper layers, 50 x 50 mm, 126 parts, among them IC1 BD62120AEFJ-E2, J1 Conn_01x05_Male, J2 Solenoid(Sol), J3 USB_C_Receptacle_USB2.0, J4 Conn_01x03_Male, J5 Conn_01x06_Male, J6 Conn_01x02_Male, J7 Endstop Switch 1, J8 Endstop Switch 2, Q1 MMDT2222A, Q2 SI2366DS, U1 ESP32-PICO-D4, U2 TPS54233D, U3 CP2102-GMR-QFN28, U4 SN65HVD230, U5 LTC4411, U6 RT9025-25GSP, U7 LTC4411

Commit message: Chad V2
Parts:
- removed C32: 160pF, Capacitor_SMD:C_0603_1608Metric
- added G***: LOGO, iclr:iclr_logo, B.Cu at (61.6, 41.8)
- C2: value 0.1uF -> 1uF
- R26, R27: value 90 -> 110
- R29, R30: footprint Resistor_SMD:R_0805_2012Metric -> Resistor_SMD:R_0603_1608Metric
- R4: value 3.5k -> 3k
- U6: value RT9025-25GSP -> SC2416H
- moved TP12 0.88 mm to (72.6, 36.7)
- moved TP11 0.16 mm to (88.4, 45.3)
- moved R29 0.11 mm to (75.4, 65.3)
- moved R30 0.10 mm to (75.4, 63.5)
Connections:
- R24 pad 2: (no net) -> Net-(R24-Pad2)
- U1 pad 10: /ServoPWM -> /ES1GPIO
- U1 pad 25: /ES1GPIO -> /ServoPWM
- U3 pad 29: unconnected-(U3-Pad29) -> GND
Routing:
- net /ES1GPIO: track 13.7 -> 31.6 mm, vias 0 -> 2
- net GND: track 19.2 -> 31.1 mm, vias 169 -> 172
- net /ServoPWM: track 27.1 -> 36.7 mm, vias 0 -> 1
- net +6V: track 36.2 -> 34.7 mm
- net /CAN_HIGH: track 23.6 -> 24.4 mm
- net +3V3: track 62.9 -> 63.4 mm
Other:
- board text added: "6V PAD"
- board text added: "C.H.A.D-v2"
- board text removed: "C.H.A.D-v1"
