File: Chad/Hardware/Actuators Board.kicad_pcb (KiCad board)
At the start: 4 copper layers, 50 x 50 mm, 126 parts, among them IC1 BD62120AEFJ-E2, J1 Conn_01x05_Male, J2 Solenoid(Sol), J3 USB_C_Receptacle_USB2.0, J4 Conn_01x03_Male, J5 Conn_01x06_Male, J6 Conn_01x02_Male, J7 Endstop Switch 1, J8 Endstop Switch 2, Q1 MMDT2222A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

Commit message: updated silkscreen, antenna line width and removed can resistors
Parts:
- removed R26, R27: 110, Resistor_SMD:R_0603_1608Metric
Connections:
- U4 pad 1: Net-(R26-Pad2) -> /CAN_TX
- U4 pad 4: Net-(R27-Pad2) -> /CAN_RX
Routing:
- net /CAN_TX: track 1.50 -> 8.07 mm
- net Net-(R26-Pad2): track 5.06 -> 0.00 mm
- net /CAN_RX: track 6.49 -> 11.0 mm
- net Net-(R27-Pad2): track 3.81 -> 0.00 mm
- net GND: vias 172 -> 173
