File: Chad/Hardware/Actuators Board.kicad_sch (KiCad schematic)
At the start: 83 parts, among them IC1 BD62120AEFJ-E2, J1 Conn_01x05_Male, J10 Conn_01x02_Male, J2 Solenoid(Sol), J4 Conn_01x03_Male, J5 Conn_01x06_Male, J6 Conn_01x02_Male, J9 Conn_01x02_Male, Q1 MMDT2222A, Q2 SI2366DS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

Commit message: changed autoprogrammer cap values
Parts:
- C2: value 1uF -> 0.1uF
- C3: value 1uF -> 1nF
Changed lines of the file:
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@@
     (in_bom yes) (on_board yes)
     (property "Reference" "C2" (id 0) (at 22.86 185.9534 90))
-    (property "Value" "1uF" (id 1) (at 22.86 188.2648 90))
+    (property "Value" "0.1uF" (id 1) (at 22.86 188.2648 90))
     (property "Footprint" "Capacitor_SMD:C_0603_1608Metric" (id 2) (at 22.86 191.77 0)
       (effects (font (size 1.27 1.27)) hide)
@@
     (in_bom yes) (on_board yes)
     (property "Reference" "C3" (id 0) (at 54.61 164.3634 90))
-    (property "Value" "1uF" (id 1) (at 54.61 166.6748 90))
+    (property "Value" "1nF" (id 1) (at 54.61 166.6748 90))
     (property "Footprint" "Capacitor_SMD:C_0603_1608Metric" (id 2) (at 54.61 170.18 0)
       (effects (font (size 1.27 1.27)) hide)
@@
     (pin "3")
     (pin "4")
-    (pin "9")
     (pin "5")
     (pin "6")
     (pin "7")
     (pin "8")
+    (pin "9")
   )
   (symbol (lib_id "power:GND") (at 250.19 85.09 0) (unit 1)
@@
     )
     (path "/00000000-0000-0000-0000-00005da70d8a"
-      (reference "C2") (unit 1) (value "1uF") (footprint "Capacitor_SMD:C_0603_1608Metric")
+      (reference "C2") (unit 1) (value "0.1uF") (footprint "Capacitor_SMD:C_0603_1608Metric")
     )
     (path "/00000000-0000-0000-0000-00005dab5946"
-      (reference "C3") (unit 1) (value "1uF") (footprint "Capacitor_SMD:C_0603_1608Metric")
+      (reference "C3") (unit 1) (value "1nF") (footprint "Capacitor_SMD:C_0603_1608Metric")
     )
     (path "/194a6401-2f3b-4426-b35d-f49a3f03a2bd"

Commit message: changed boot and EN jumper Caps
Parts:
- C1: value 1uF -> 0.1uF
- C3: value 1nF -> 0.1uF
Changed lines of the file:
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@@
     (in_bom yes) (on_board yes)
     (property "Reference" "C3" (id 0) (at 54.61 164.3634 90))
-    (property "Value" "1nF" (id 1) (at 54.61 166.6748 90))
+    (property "Value" "0.1uF" (id 1) (at 54.61 166.6748 90))
     (property "Footprint" "Capacitor_SMD:C_0603_1608Metric" (id 2) (at 54.61 170.18 0)
       (effects (font (size 1.27 1.27)) hide)
@@
     (in_bom yes) (on_board yes)
     (property "Reference" "C1" (id 0) (at 25.4 164.3634 90))
-    (property "Value" "1uF" (id 1) (at 25.4 166.6748 90))
+    (property "Value" "0.1uF" (id 1) (at 25.4 166.6748 90))
     (property "Footprint" "Capacitor_SMD:C_0603_1608Metric" (id 2) (at 25.4 170.18 0)
       (effects (font (size 1.27 1.27)) hide)
@@
     )
     (path "/00000000-0000-0000-0000-00005dabbfe7"
-      (reference "C1") (unit 1) (value "1uF") (footprint "Capacitor_SMD:C_0603_1608Metric")
+      (reference "C1") (unit 1) (value "0.1uF") (footprint "Capacitor_SMD:C_0603_1608Metric")
     )
     (path "/00000000-0000-0000-0000-00005da70d8a"
@@
     )
     (path "/00000000-0000-0000-0000-00005dab5946"
-      (reference "C3") (unit 1) (value "1nF") (footprint "Capacitor_SMD:C_0603_1608Metric")
+      (reference "C3") (unit 1) (value "0.1uF") (footprint "Capacitor_SMD:C_0603_1608Metric")
     )
     (path "/194a6401-2f3b-4426-b35d-f49a3f03a2bd"

Commit message: Implemented design review feedback
Parts:
- removed TP22, TP25: TestPoint, TestPoint:TestPoint_Pad_D1.5mm, symbol Connector:TestPoint
- added J7: Endstop Switch 1, TestPoint:TestPoint_Pad_D1.5mm, symbol Connector:Conn_01x01_Female
- added J8: Endstop Switch 2, TestPoint:TestPoint_Pad_D1.5mm, symbol Connector:Conn_01x01_Female
- 3V3LED1: renamed from D6; value PWR_LED -> 3V3LED
- L2: value ETQP5M -> 33uH
- renumbered D7 to 24VLED1, J10 to BOOTJUMPER1, J9 to ENJUMPER1, D2 to RXLED1, D1 to SolLED1, D3 to TXLED1
Connections:
- net ES1GPIO: now also J7.1 (Pin_1)
- net ES2GPIO: now also J8.1 (Pin_1)
Other:
- note added: "And only add this resistor to pull-down the SSR pin"
- note added: "Only add this resistor to pull-up the SSR pin"
- note added: "Otherwise, do not add either resistor for microcontroller output. This would've been a solder jumper, but PCB space is a luxury."
- moved on the sheet: R32

Commit message: Chad V2
Parts:
- C2: value 0.1uF -> 1uF
- R4: value 3.5k -> 3k
Connections:
- net ES1GPIO: now also U1.10 (IO34); no longer U1.25 (IO16)
- net ServoPWM: now also U1.25 (IO16); no longer U1.10 (IO34)
Changed lines of the file:
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@@
     (stroke (width 0) (type default) (color 0 0 0 0))
   )
+  (wire (pts (xy 83.82 96.52) (xy 93.98 96.52))
+    (stroke (width 0) (type default) (color 0 0 0 0))
+  )
   (wire (pts (xy 93.98 54.61) (xy 95.25 54.61))
     (stroke (width 0) (type default) (color 0 0 0 0))
@@
     (stroke (width 0) (type default) (color 0 0 0 0))
   )
+  (wire (pts (xy 134.62 121.92) (xy 143.51 121.92))
+    (stroke (width 0) (type default) (color 0 0 0 0))
+  )
   (wire (pts (xy 92.71 27.94) (xy 92.71 26.67))
     (stroke (width 0) (type default) (color 0 0 0 0))
@@
     (stroke (width 0) (type default) (color 0 0 0 0))
   )
-  (wire (pts (xy 134.62 121.92) (xy 144.78 121.92))
-    (stroke (width 0) (type default) (color 0 0 0 0))
-  )
   (wire (pts (xy 134.62 114.3) (xy 143.51 114.3))
     (stroke (width 0) (type default) (color 0 0 0 0))
@@
     (effects (font (size 1.27 1.27)) (justify right bottom))
   )
-  (label "ServoPWM" (at 144.78 121.92 180)
-    (effects (font (size 1.27 1.27)) (justify right bottom))
-  )
   (label "Hall1" (at 143.51 116.84 180)
     (effects (font (size 1.27 1.27)) (justify right bottom))
@@
     (effects (font (size 1.27 1.27)) (justify right bottom))
   )
+  (label "ServoPWM" (at 93.98 96.52 180)
+    (effects (font (size 1.27 1.27)) (justify right bottom))
+  )
   (label "CAN_RX" (at 143.51 114.3 180)
     (effects (font (size 1.27 1.27)) (justify right bottom))
@@
     (effects (font (size 1.27 1.27)) (justify right bottom))
   )
-  (label "ES1GPIO" (at 93.98 96.52 180)
-    (effects (font (size 1.27 1.27)) (justify right bottom))
-  )
   (label "RXD" (at 17.78 21.59 0)
     (effects (font (size 1.27 1.27)) (justify left bottom))
@@
     (effects (font (size 1.27 1.27)) (justify right bottom))
   )
+  (label "ES1GPIO" (at 143.51 121.92 180)
+    (effects (font (size 1.27 1.27)) (justify right bottom))
+  )
   (label "RXD" (at 143.51 68.58 180)
     (effects (font (size 1.27 1.27)) (justify right bottom))
@@
     (in_bom yes) (on_board yes)
     (property "Reference" "C2" (id 0) (at 22.86 185.9534 90))
-    (property "Value" "0.1uF" (id 1) (at 22.86 188.2648 90))
+    (property "Value" "1uF" (id 1) (at 22.86 188.2648 90))
     (property "Footprint" "Capacitor_SMD:C_0603_1608Metric" (id 2) (at 22.86 191.77 0)
       (effects (font (size 1.27 1.27)) hide)
@@
     (in_bom yes) (on_board yes)
     (property "Reference" "R4" (id 0) (at 68.58 21.6916 90))
-    (property "Value" "3.5k" (id 1) (at 68.58 24.003 90))
+    (property "Value" "3k" (id 1) (at 68.58 24.003 90))
     (property "Footprint" "Resistor_SMD:R_0603_1608Metric" (id 2) (at 68.58 26.67 0)
       (effects (font (size 1.27 1.27)) hide)
@@
     (pin "2")
   )
+  (symbol (lib_id "Connector:TestPoint") (at 83.82 96.52 90) (unit 1)
+    (in_bom yes) (on_board yes)
+    (property "Reference" "TP12" (id 0) (at 79.0448 97.6884 90)
+      (effects (font (size 1.27 1.27)) (justify left))
+    )
+    (property "Value" "TestPoint" (id 1) (at 79.0448 95.377 90)
+      (effects (font (size 1.27 1.27)) (justify left))
+    )
+    (property "Footprint" "TestPoint:TestPoint_Pad_D1.0mm" (id 2) (at 83.82 91.44 0)
+      (effects (font (size 1.27 1.27)) hide)
+    )
+    (property "Datasheet" "~" (id 3) (at 83.82 91.44 0)
+      (effects (font (size 1.27 1.27)) hide)
+    )
+    (pin "1")
+  )
   (symbol (lib_id "iclr:BD62120AEFJ-E2") (at 205.74 82.55 0) (unit 1)
     (in_bom yes) (on_board yes) (fields_autoplaced)
@@
     (pin "1")
   )
-  (symbol (lib_id "Connector:TestPoint") (at 144.78 121.92 270) (unit 1)
-    (in_bom yes) (on_board yes)
-    (property "Reference" "TP12" (id 0) (at 149.5552 120.7516 90)
-      (effects (font (size 1.27 1.27)) (justify left))
-    )
-    (property "Value" "TestPoint" (id 1) (at 149.5552 123.063 90)
-      (effects (font (size 1.27 1.27)) (justify left))
-    )
-    (property "Footprint" "TestPoint:TestPoint_Pad_D1.0mm" (id 2) (at 144.78 127 0)
-      (effects (font (size 1.27 1.27)) hide)
-    )
-    (property "Datasheet" "~" (id 3) (at 144.78 127 0)
-      (effects (font (size 1.27 1.27)) hide)
-    )
-    (pin "1")
-  )
   (symbol (lib_id "Device:C_Small") (at 95.25 49.53 0) (unit 1)
     (in_bom yes) (on_board yes)
@@
       (reference "#PWR0114") (unit 1) (value "GND") (footprint "")
     )
+    (path "/00000000-0000-0000-0000-000061925999/c9a8b450-3b80-4c73-8844-e1ff92c5c260"
+      (reference "#PWR0115") (unit 1) (value "GND") (footprint "")
+    )
     (path "/0b72ffc6-666f-4365-a8e2-e330a45de594"
       (reference "#PWR0116") (unit 1) (value "GND") (footprint "")
@@
     )
     (path "/00000000-0000-0000-0000-00005da70d8a"
-      (reference "C2") (unit 1) (value "0.1uF") (footprint "Capacitor_SMD:C_0603_1608Metric")
+      (reference "C2") (unit 1) (value "1uF") (footprint "Capacitor_SMD:C_0603_1608Metric")
     )
     (path "/00000000-0000-0000-0000-00005dab5946"
@@
       (reference "C31") (unit 1) (value "0.1uF") (footprint "Capacitor_SMD:C_0603_1608Metric")
     )
-    (path "/00000000-0000-0000-0000-000061942b9a/39194db9-a03c-43f0-ad59-d69dd5910874"
-      (reference "C32") (unit 1) (value "160pF") (footprint "Capacitor_SMD:C_0603_1608Metric")
-    )
     (path "/00000000-0000-0000-0000-000061942b9a/759646bf-5c31-420e-aff7-2c1a28ce32e1"
       (reference "C33") (unit 1) (value "100nF") (footprint "Capacitor_SMD:C_0603_1608Metric")
@@
     )
     (path "/00000000-0000-0000-0000-000061b6bc0b"
-      (reference "R4") (unit 1) (value "3.5k") (footprint "Resistor_SMD:R_0603_1608Metric")
+      (reference "R4") (unit 1) (value "3k") (footprint "Resistor_SMD:R_0603_1608Metric")
     )
     (path "/00000000-0000-0000-0000-00005dabbfed"
@@
     )
     (path "/00000000-0000-0000-0000-000061942b9a/4ebf59df-bc69-439f-b9f2-cb433efbca66"
-      (reference "R26") (unit 1) (value "90") (footprint "Resistor_SMD:R_0603_1608Metric")
+      (reference "R26") (unit 1) (value "110") (footprint "Resistor_SMD:R_0603_1608Metric")
     )
     (path "/00000000-0000-0000-0000-000061942b9a/476229cc-ca1e-4a0f-8f09-96ad5be435cb"
-      (reference "R27") (unit 1) (value "90") (footprint "Resistor_SMD:R_0603_1608Metric")
+      (reference "R27") (unit 1) (value "110") (footprint "Resistor_SMD:R_0603_1608Metric")
     )
     (path "/00000000-0000-0000-0000-000061942b9a/c0a35b75-0e83-4311-add3-5a3930110d30"
@@
     )
     (path "/00000000-0000-0000-0000-000061942b9a/c4e42d16-8dbe-42af-a61a-faa72b95fe53"
-      (reference "R29") (unit 1) (value "60") (footprint "Resistor_SMD:R_0805_2012Metric")
+      (reference "R29") (unit 1) (value "60") (footprint "Resistor_SMD:R_0603_1608Metric")
     )
     (path "/00000000-0000-0000-0000-000061942b9a/c363df37-be76-44cd-846e-5e1010ee0d3e"
-      (reference "R30") (unit 1) (value "60") (footprint "Resistor_SMD:R_0805_2012Metric")
+      (reference "R30") (unit 1) (value "60") (footprint "Resistor_SMD:R_0603_1608Metric")
     )
     (path "/116e1149-ba9e-462a-beb7-8e276ef3a596"
@@
       (reference "TP11") (unit 1) (value "TestPoint") (footprint "TestPoint:TestPoint_Pad_D1.0mm")
     )
-    (path "/f8a7cf99-fb92-4312-b900-3804c63ab7dd"
+    (path "/a101baee-116e-4be1-9a34-0dfd37bf6955"
       (reference "TP12") (unit 1) (value "TestPoint") (footprint "TestPoint:TestPoint_Pad_D1.0mm")
     )
@@
     )
     (path "/00000000-0000-0000-0000-000061925999/a8f5718a-9498-4816-a1ce-ace2140e0f78"
-      (reference "U6") (unit 1) (value "RT9025-25GSP") (footprint "iclr:SOIC127P599X175-9N")
+      (reference "U6") (unit 1) (value "SC2416H") (footprint "iclr:SOIC127P599X175-9N")
     )
     (path "/00000000-0000-0000-0000-000061925999/261fd709-b119-45e9-aff5-04154ebd9314"
