File: Chad/Hardware/can.kicad_sch (KiCad schematic)
At the start: 14 parts, among them U4 SN65HVD230

Commit message: Chad V2
Parts:
- removed C32: 160pF, Capacitor_SMD:C_0603_1608Metric, symbol Device:C_Small
- R26, R27: value 90 -> 110
- R29, R30: footprint Resistor_SMD:R_0805_2012Metric -> Resistor_SMD:R_0603_1608Metric
Changed lines of the file:
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@@
   (junction (at 156.21 80.01) (diameter 0) (color 0 0 0 0)
   )
-  (junction (at 118.11 85.09) (diameter 0) (color 0 0 0 0)
-  )
   (junction (at 129.54 68.58) (diameter 0) (color 0 0 0 0)
   )
   (junction (at 163.83 88.9) (diameter 0) (color 0 0 0 0)
   )
-  (junction (at 124.46 97.79) (diameter 0) (color 0 0 0 0)
-  )
   (junction (at 156.21 97.79) (diameter 0) (color 0 0 0 0)
   )
@@
     (stroke (width 0) (type default) (color 0 0 0 0))
   )
-  (wire (pts (xy 118.11 90.17) (xy 118.11 97.79))
-    (stroke (width 0) (type default) (color 0 0 0 0))
-  )
-  (wire (pts (xy 118.11 97.79) (xy 124.46 97.79))
-    (stroke (width 0) (type default) (color 0 0 0 0))
-  )
   (wire (pts (xy 124.46 73.66) (xy 127 73.66))
     (stroke (width 0) (type default) (color 0 0 0 0))
@@
     (stroke (width 0) (type default) (color 0 0 0 0))
   )
-  (wire (pts (xy 118.11 85.09) (xy 124.46 85.09))
-    (stroke (width 0) (type default) (color 0 0 0 0))
-  )
-  (wire (pts (xy 116.84 85.09) (xy 118.11 85.09))
+  (wire (pts (xy 116.84 85.09) (xy 124.46 85.09))
     (stroke (width 0) (type default) (color 0 0 0 0))
   )
@@
     (pin "2")
   )
-  (symbol (lib_id "Device:C_Small") (at 118.11 87.63 180) (unit 1)
-    (in_bom yes) (on_board yes)
-    (property "Reference" "C32" (id 0) (at 119.38 81.28 0)
-      (effects (font (size 1.27 1.27)) (justify right))
-    )
-    (property "Value" "160pF" (id 1) (at 118.11 83.82 0)
-      (effects (font (size 1.27 1.27)) (justify right))
-    )
-    (property "Footprint" "Capacitor_SMD:C_0603_1608Metric" (id 2) (at 118.11 87.63 0)
-      (effects (font (size 1.27 1.27)) hide)
-    )
-    (property "Datasheet" "~" (id 3) (at 118.11 87.63 0)
-      (effects (font (size 1.27 1.27)) hide)
-    )
-    (pin "1")
-    (pin "2")
-  )
   (symbol (lib_id "Diode:SM712_SOT23") (at 175.26 88.9 270) (unit 1)
     (in_bom yes) (on_board yes)
@@
     (in_bom yes) (on_board yes)
     (property "Reference" "R27" (id 0) (at 114.3 90.17 90))
-    (property "Value" "90" (id 1) (at 114.3 92.71 90))
+    (property "Value" "110" (id 1) (at 114.3 92.71 90))
     (property "Footprint" "Resistor_SMD:R_0603_1608Metric" (id 2) (at 114.3 87.63 0)
       (effects (font (size 1.27 1.27)) hide)
@@
     (in_bom yes) (on_board yes)
     (property "Reference" "R26" (id 0) (at 114.3 80.01 90))
-    (property "Value" "90" (id 1) (at 114.3 82.55 90))
+    (property "Value" "110" (id 1) (at 114.3 82.55 90))
     (property "Footprint" "Resistor_SMD:R_0603_1608Metric" (id 2) (at 114.3 85.09 0)
       (effects (font (size 1.27 1.27)) hide)
@@
       (effects (font (size 1.27 1.27)) (justify left))
     )
-    (property "Footprint" "Resistor_SMD:R_0805_2012Metric" (id 2) (at 154.432 93.98 90)
+    (property "Footprint" "Resistor_SMD:R_0603_1608Metric" (id 2) (at 154.432 93.98 90)
       (effects (font (size 1.27 1.27)) hide)
     )
@@
       (effects (font (size 1.27 1.27)) (justify left))
     )
-    (property "Footprint" "Resistor_SMD:R_0805_2012Metric" (id 2) (at 154.432 83.82 90)
-      (effects (font (size 1.27 1.27)) hide)
-    )
+    (property "Footprint" "Resistor_SMD:R_0603_1608Metric" (id 2) (at 154.432 83.82 90)
+      (effects (font (size 1.27 1.27)) hide)
+    )

Commit message: updated silkscreen, antenna line width and removed can resistors
Parts:
- removed R26, R27: 110, Resistor_SMD:R_0603_1608Metric, symbol Device:R_Small
Connections:
- net CAN_RX: now also U4.4 (R)
- net CAN_TX: now also U4.1 (D)
Changed lines of the file:
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@@
     (stroke (width 0) (type default) (color 0 0 0 0))
   )
-  (wire (pts (xy 116.84 87.63) (xy 124.46 87.63))
+  (wire (pts (xy 111.76 87.63) (xy 124.46 87.63))
     (stroke (width 0) (type default) (color 0 0 0 0))
   )
@@
     (stroke (width 0) (type default) (color 0 0 0 0))
   )
-  (wire (pts (xy 116.84 85.09) (xy 124.46 85.09))
+  (wire (pts (xy 111.76 85.09) (xy 124.46 85.09))
     (stroke (width 0) (type default) (color 0 0 0 0))
   )
@@
     (pin "3")
   )
-  (symbol (lib_id "Device:R_Small") (at 114.3 87.63 90) (unit 1)
-    (in_bom yes) (on_board yes)
-    (property "Reference" "R27" (id 0) (at 114.3 90.17 90))
-    (property "Value" "110" (id 1) (at 114.3 92.71 90))
-    (property "Footprint" "Resistor_SMD:R_0603_1608Metric" (id 2) (at 114.3 87.63 0)
-      (effects (font (size 1.27 1.27)) hide)
-    )
-    (property "Datasheet" "~" (id 3) (at 114.3 87.63 0)
-      (effects (font (size 1.27 1.27)) hide)
-    )
-    (pin "1")
-    (pin "2")
-  )
   (symbol (lib_id "power:GND") (at 163.83 88.9 0) (unit 1)
     (in_bom yes) (on_board yes) (fields_autoplaced)
@@
     (pin "1")
   )
-  (symbol (lib_id "Device:R_Small") (at 114.3 85.09 90) (unit 1)
-    (in_bom yes) (on_board yes)
-    (property "Reference" "R26" (id 0) (at 114.3 80.01 90))
-    (property "Value" "110" (id 1) (at 114.3 82.55 90))
-    (property "Footprint" "Resistor_SMD:R_0603_1608Metric" (id 2) (at 114.3 85.09 0)
-      (effects (font (size 1.27 1.27)) hide)
-    )
-    (property "Datasheet" "~" (id 3) (at 114.3 85.09 0)
-      (effects (font (size 1.27 1.27)) hide)
-    )
-    (pin "1")
-    (pin "2")
-  )
   (symbol (lib_id "power:GND") (at 163.83 102.87 0) (unit 1)
