File: Hardware/Chad.kicad_sch (KiCad schematic)
At the start: 60 parts, among them J1 RBUS, J2 ServoCH2, J4 ServoCH1, J7 Endstop Switch 1, J8 Endstop Switch 2, U1 ESP32-S3, U2 TPS54233D, U5 LTC4411

Commit message: added jumper to change the buck converter to 8.4v
Parts:
- removed R10: 470, Resistor_SMD:R_0603_1608Metric, symbol Device:R_Small
- removed RXLED1: RX_LED, LED_SMD:LED_0603_1608Metric, symbol Device:LED_Small
- added C26: 10uF, Capacitor_SMD:C_0603_1608Metric, symbol Device:C_Small
- added JP3: AltVJP, Jumper:SolderJumper-2_P1.3mm_Open_RoundedPad1.0x1.5mm, symbol Jumper:SolderJumper_2_Open
- added R2: 3.3K, Resistor_SMD:R_0603_1608Metric, symbol Device:R_Small
- C1, C13, C15, C16, C2, C22, C3, C6: footprint Capacitor_SMD:C_0603_1608Metric -> Capacitor_SMD:C_0402_1005Metric
- C10, C11, C7, C8, C9: renamed from C?; footprint (none) -> Capacitor_SMD:C_0402_1005Metric
- C12, C17, C18, C21, C24: renamed from C?; footprint Capacitor_SMD:C_0603_1608Metric -> Capacitor_SMD:C_0402_1005Metric
- C14: footprint Capacitor_SMD:C_1210_3225Metric -> Capacitor_SMD:C_0603_1608Metric
- C5: renamed from C?; footprint (none) -> Capacitor_SMD:C_0603_1608Metric
- JP2: renamed from JP?; footprint (none) -> Jumper:SolderJumper-2_P1.3mm_Open_RoundedPad1.0x1.5mm
- R1: renamed from R?; footprint (none) -> Resistor_SMD:R_0402_1005Metric
- Y1: renamed from Y?; footprint (none) -> Crystal:Crystal_SMD_2016-4Pin_2.0x1.6mm
- gave numbers to parts that had none: 2
Connections:
- net GND: now also C26.1, R2.2
- net VSENSE: now also JP3.1 (A)
- net at J1.3 (Pin_3), U5.1 (IN): now also C26.2
- new net: JP3.2 (B), R2.1
Other:
- note added: "Bridge this jumper to switch the buck to the alternate voltage. With a 3.3K resistor, the this voltage is 8.4V"
- moved on the sheet: R11, TXLED1
