File: Hardware/Chad.kicad_sch (KiCad schematic)
At the start: 58 parts, among them J1 RBUS, J2 GPIO Breakout, J3 ServoCH1, J4 ServoCH2, U1 ESP32-S3, Y1 40MHz±10ppm

Commit message: crystal and caps
Parts:
- C12: value 4.2pF -> DNP
- C13, C14: value C -> 11pF
- R5: value 47.5 -> DNP
- Y1: value 40MHz±10ppm -> R940000171
Changed lines of the file:
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@@
     (stroke (width 0) (type default))
+  )
+  (text_box "Crystal must be 40 MHz and at least ±10ppm"
+    (at 144.78 147.32 0) (size 19.05 11.43)
+    (stroke (width -0.0001) (type default))
+    (fill (type none))
+    (effects (font (size 1.27 1.27)) (justify left top))
   )
   (text_box "Optional pull-up resistors for the broken out GPIOs."
@@
       (effects (font (size 1.27 1.27)) (justify left))
     )
-    (property "Value" "C" (at 165.1 144.5514 90)
+    (property "Value" "11pF" (at 165.1 144.5514 90)
       (effects (font (size 1.27 1.27)) (justify left))
     )
@@
       (effects (font (size 1.27 1.27)) (justify left))
     )
-    (property "Value" "C" (at 163.83 124.2314 90)
+    (property "Value" "11pF" (at 163.83 124.2314 90)
       (effects (font (size 1.27 1.27)) (justify left))
     )
@@
       (effects (font (size 1.27 1.27)) (justify left))
     )
-    (property "Value" "4.2pF" (at 68.58 59.69 90)
+    (property "Value" "DNP" (at 68.58 59.69 90)
       (effects (font (size 1.27 1.27)) (justify left))
     )
@@
   (symbol (lib_id "Device:Crystal_GND24") (at 156.21 132.08 90) (unit 1)
     (in_bom yes) (on_board yes) (dnp no)
-    (property "Reference" "Y1" (at 152.4 121.92 90)
-      (effects (font (size 1.27 1.27)))
-    )
-    (property "Value" "40MHz±10ppm" (at 152.4 124.46 90)
+    (property "Reference" "Y1" (at 149.86 121.92 90)
+      (effects (font (size 1.27 1.27)))
+    )
+    (property "Value" "R940000171" (at 149.86 124.46 90)
       (effects (font (size 1.27 1.27)))
     )
@@
       (effects (font (size 1.27 1.27)))
     )
-    (property "Value" "47.5" (at 57.15 59.69 90)
-      (effects (font (size 1.27 1.27)))
-    )
+    (property "Value" "DNP" (at 57.15 59.69 90)
+      (effects (font (size 1.27 1.27)))
+    )
