File: Hardware/buckC.kicad_sch (KiCad schematic)
At the start: 33 parts, among them Q1 SSM3K15AMFV,L3F, U6 SiC437BED-T1-GE3

Commit message: changed inductor to one that won't heat up as much
Parts:
- L4: footprint iclr:EXL1V07053R3R -> iclr:IND_SPM10065VT-3R3M-D
Other:
- note added: "SPM10065VT-3R3M-D"
- note removed: "EXL1V0705-3R3-R"
Changed lines of the file:
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@@
     (effects (font (size 1.27 1.27)) (justify left bottom))
   )
-  (text "EXL1V0705-3R3-R" (at 54.61 68.58 0)
+  (text "SPM10065VT-3R3M-D" (at 50.8 68.58 0)
     (effects (font (size 1.27 1.27)) (justify left bottom))
   )
@@
       (effects (font (size 1.27 1.27)))
     )
-    (property "Footprint" "iclr:EXL1V07053R3R" (at 67.31 66.04 0)
-      (effects (font (size 1.27 1.27)) hide)
-    )
+    (property "Footprint" "iclr:IND_SPM10065VT-3R3M-D" (at 67.31 66.04 0)
+      (effects (font (size 1.27 1.27)) hide)
+    )
